File: render/illustration/esp32s3-camera-illustration.kicad_pcb (KiCad board)
At the start: 4 copper layers, 60 x 85 mm, 69 parts, among them J1 USB-C, J2 OV2640/OV5640 24P, J3 microSD, J4 LiPo 3.7V, J5 UART / DEBUG, J6 EXPANSION, Q1 AO3400A, Q2 AO3401A, SW1 BOOT, SW2 RESET, SW3 SHUTTER, SW4 PWR, U1 ESP32-S3-WROOM-1-N16R8, U2 AP2112K-3.3, U3 TP4056, U4 USBLC6-2SC6, U5 XC6206P282MR, U6 XC6206P122MR

Commit message: Board v1.4: side-actuated shutter on the top edge
SW3 SHUTTER moves from the lens face (top-actuated SKQG at 9,40) to an
ALPS SKRTLAE010 side switch at (50.6, 2.6) with the stem pointing off the
top edge, so the enclosure's top wall can carry the shutter button under
the right index finger. Project footprint copy with 0.55 mm pads for hole
clearance, SolidWorks-made simplified STEP model (KiCad's library has
none), C12 moved 0.8 mm, BTN_SHUTTER rerouted under the module (B.Cu
y 73.4) and up the right edge (x 59.35). ERC 0, DRC with parity 0/0/0,
GND/3V3 connectivity 0 isolated pads; CPL differs from v1.3 only in C12
and SW3. Fab outputs, versions/v1.4 snapshot, renders and docs updated.

Co-Authored-By: Claude Fable 5.1 <noreply@anthropic.com>
Parts:
- removed J6: EXPANSION, Connector_PinHeader_2.54mm:PinHeader_1x04_P2.54mm_Vertical
- D5: footprint LED_0603_1608Metric -> LED_SMD:LED_0603_1608Metric
- J5: value UART / DEBUG -> DISPLAY 1.3in ST7789; footprint Connector_PinHeader_2.54mm:PinHeader_1x04_P2.54mm_Vertical -> Connector_PinSocket_2.54mm:PinSocket_1x07_P2.54mm_Vertical
- R20, R21: footprint R_0603_1608Metric -> Resistor_SMD:R_0603_1608Metric
- SW3: footprint Button_Switch_SMD:SW_SPST_SKQG_WithoutStem -> esp32s3-camera:SW_Push_SKRTLAE010_Side
- SW4: footprint SW_SPDT_Shouhan_MSK12C02 -> Button_Switch_SMD:SW_SPDT_Shouhan_MSK12C02
- moved SW3 55.9 mm to (50.6, 2.60), turned to 180 degrees
- moved J5 12.6 mm to (56.0, 52.6), turned to 0 degrees
- moved ILL4 4.89 mm to (38.9, 45.0)
- moved C12 0.80 mm to (47.5, 6.30)
- turned R21 to -90 degrees
Connections:
- J5 pad 1: +3V3 -> GND
- J5 pad 2: GND -> +3V3
- J5 pad 3: UART_TX -> UART_RX
- J5 pad 4: UART_RX -> UART_TX
- R21 pad 1: LDO_EN -> VSYS
- R21 pad 2: VSYS -> LDO_EN
- SW4 pad 1: (no net) -> unconnected-(SW4-A-Pad1)
Routing:
- net BTN_SHUTTER: track 77.8 -> 159.5 mm, vias 1 -> 3
- net IO4: track 23.0 -> 48.9 mm, vias 2 -> 3
- net IO6: track 19.6 -> 41.5 mm, vias 0 -> 1
- net IO5: track 24.9 -> 46.6 mm, vias 0 -> 1
- net GND: track 39.7 -> 45.3 mm, vias 184 -> 183
- net IPROG: track 26.8 -> 27.5 mm
- net +3V3: track 27.1 -> 27.7 mm
Other:
- board text added: "1.3in ST7789 module 27.78 x 39.22, plugs into J5"
- board text added: "3V3"
- board text added: "BLK"
- board text added: "DC"
- board text added: "DISPLAY"
- board text added: "ESP32-S3 CAMERA v1.4"
- board text added: "GND"
- board text added: "RES"
- board text added: "SCL"
- board text added: "SDA"
- board text added: "SHUTTER"
- board text removed: "ESP32-S3 CAMERA v1.2"
